File: gps/skycan-gps.sch (KiCad schematic (older format))
At the start: 6 parts, among them J1 SMA, U1 Taoglas CGGP.25.A

Commit message: GPS layout finished.
Connections:
- net SGNL: now reaches J1.1 (RF), U1.1 (S)
Changed lines of the file:
@@
 Wire Wire Line
 	6350 6100 6350 6350
+Text Label 8050 5950 1    60   ~ 0
+SGNL
 $EndSCHEMATC

Commit message: Added SMA Farnell code sch.
Parts:
- J1: Farnell (none) -> 1248990
Changed lines of the file:
@@
 F 2 "SMA" H 8400 6300 50  0001 C CNN
 F 3 "" H 8200 6300 60  0000 C CNN
+F 4 "1248990" H 8200 6300 60  0001 C CNN "Farnell"
 	1    8200 6300
 	1    0    0    -1
